File: hardware/openRiverSense_010/openRiverSense_010.kicad_sch (KiCad schematic)
At the start: 0 parts

Commit message: setup KiCad
Parts:
- added C1, C2: 0402,1.5pF,50V,C0G, Capacitor_SMD:C_0402_1005Metric, symbol jlcpcb-basic-capacitor:0402,1.5pF,50V,C0G
- added C3: TAJA106K016RNJ, footprint:CAP-SMD_L3.2-W1.6-RD-C7171, symbol jlcpcb-tantalum-capacitors:TAJA106K016RNJ
- added JP1: Jumper_2_Bridged, TestPoint:TestPoint_2Pads_Pitch5.08mm_Drill1.3mm, symbol Jumper:Jumper_2_Bridged
- added L1: CMI201209U2R2KT, footprint:L0805, symbol jlcpcb-inductors-ferrite-beads:CMI201209U2R2KT
- added LED1: 19-217_GHC-YR1S2_3T, footprint:LED0603-RD, symbol jlcpcb-diodes:19-217_GHC-YR1S2_3T
- added R1: 0402,0, Resistor_SMD:R_0402_1005Metric, symbol jlcpcb-basic-resistor:0402,0
- added U1: B5819W_C8598, footprint:SOD-123_L2.7-W1.6-LS3.7-RD-1, symbol jlcpcb-diodes:B5819W_C8598
- added U2: MCP6002T-I_SN, footprint:SOIC-8_L4.9-W3.9-P1.27-LS6.0-BL, symbol jlcpcb-analog:MCP6002T-I_SN
- added U3: PCF8563T_5,518, footprint:SOIC-8_L5.0-W4.0-P1.27-LS6.0-BL, symbol jlcpcb-chips-crystals:PCF8563T_5,518
- added U4: ESP32-S3-MINI-1U-N8, footprint:BULETM-SMD_ESPRESSIF_ESP32-S3-MINI-1U-N8, symbol jlcpcb-extended:ESP32-S3-MINI-1U-N8
- added U5: XC6220B331MR-G, footprint:SOT-25_L3.0-W1.6-P0.95-LS2.8-TL, symbol jlcpcb-extended:XC6220B331MR-G
- added U6: XC6206P332MR, footprint:SOT-23-3_L2.9-W1.6-P1.90-LS2.8-BR, symbol jlcpcb-power:XC6206P332MR
- added U7: TS-1187A-B-A-B, footprint:SW-SMD_4P-L5.1-W5.1-P3.70-LS6.5-TL-2, symbol jlcpcb-switches:TS-1187A-B-A-B
- added U8: AO3401A, footprint:SOT-23_L2.9-W1.3-P1.90-LS2.4-BR, symbol jlcpcb-transistors:AO3401A
- added U9: GT-USB-7010ASV, footprint:USB-C-SMD_G-SWITCH_GT-USB-7010ASV, symbol jlcpcb-extended:GT-USB-7010ASV
