File: hardware/openRiverSense/openRiverSense.kicad_pcb (KiCad board)
At the start: 2 copper layers, 100 x 38 mm, 110 parts, among them P1 USB-C, P2 JSTSH_01x06_Vertical, P3 JSTSH_01x06_Vertical, SW1 Reset, SW2 UP_Button, SW3 ENTER_Button, SW4 DOWN_Button, U1 AO3400A, U2 AO3401A, U3 ATGM332D-5N31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

Commit message: -added CAD models -moved to KiCAD 8.0 -clang formatting -rebuild sensor calibration -add logging and analytics file -added adaptive backlight -added work hours for gps sync
Other:
- board text added: "Compact Battery Charger to lower EMI"
- board text added: "ESD Diode for antenna?"
- board text added: "Exposed Copper under Antenna?"
- board text added: "Fix lables"
- board text added: "Larger Anular Ring to make soldering easier"
- board text added: "Larger Coincell Battery?"
- board text added: "Narrower Pads"
- board text added: "RF shield?"
- board text added: "Swap Probe and Battery Connector Locations"
- board text added: "Test Integrated Coin Cell Charger"
